File: pcbDesign/exMoudle/exMoudle.kicad_pcb (KiCad board)
At the start: 2 copper layers, 56 x 133 mm, 23 parts, among them J1 luat-esp32-s3_socket, J2 face recognition, J3 Lidar, SW1 SW_Push, SW10 SW_Push, SW11 SW_Push, SW12 SW_Push, SW2 SW_Push, SW3 SW_Push, SW4 SW_Push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

Commit message: uodate exModule pcb keyboard
Connections:
- J1 pad 10: Net-(J1-GPIO8) -> /key3
- J1 pad 11: Net-(J1-GPIO9) -> /key0
- J1 pad 24: Net-(J1-GPIO13) -> /key2
- J1 pad 27: Net-(J1-GPIO12) -> /key1
- R1 pad 1: Net-(J1-GPIO9) -> /key0
- R2 pad 2: Net-(J1-GPIO12) -> /key1
- R3 pad 2: Net-(J1-GPIO13) -> /key2
- R4 pad 1: Net-(J1-GPIO8) -> /key3
- SW1 pad 1: unconnected-(SW1-Pad1) -> /key0
- SW10 pad 1: unconnected-(SW10-Pad1) -> /key1
- SW11 pad 1: unconnected-(SW11-Pad1) -> /key2
- SW12 pad 1: unconnected-(SW12-Pad1) -> /key3
- SW2 pad 1: unconnected-(SW2-Pad1) -> /key1
- SW3 pad 1: unconnected-(SW3-Pad1) -> /key2
- SW4 pad 1: unconnected-(SW4-Pad1) -> /key3
- SW5 pad 1: unconnected-(SW5-Pad1) -> /key0
- SW6 pad 1: unconnected-(SW6-Pad1) -> /key1
- SW7 pad 1: unconnected-(SW7-Pad1) -> /key2
- SW8 pad 1: unconnected-(SW8-Pad1) -> /key3
- SW9 pad 1: unconnected-(SW9-Pad1) -> /key0
Routing:
- net /key2: track 0.00 -> 192.7 mm, vias 0 -> 2
- net /key1: track 0.00 -> 174.7 mm, vias 0 -> 5
- net /key3: track 0.00 -> 144.5 mm, vias 0 -> 5
- net /key0: track 0.00 -> 143.7 mm, vias 0 -> 1
- net Net-(J1-GPIO9): track 48.5 -> 0.00 mm
- net Net-(J1-GPIO13): track 29.3 -> 0.00 mm
- net Net-(J1-GPIO8): track 27.7 -> 0.00 mm
- net Net-(J1-GPIO12): track 19.8 -> 0.00 mm
