File: pcbDesign/exMoudle/exMoudle.kicad_sch (KiCad schematic)
At the start: 19 parts, among them J1 luat-esp32-s3_socket, J2 face recognition, J3 Lidar, SW1 SW_Push, SW10 SW_Push, SW11 SW_Push, SW12 SW_Push, SW2 SW_Push, SW3 SW_Push, SW4 SW_Push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

Commit message: uodate exModule pcb keyboard
Connections:
- net key3: now reaches SW4.1
- net key3: now also J1.10 (GPIO8), R4.1, SW12.1, SW8.1
- net key1: now reaches SW6.1
- net key1: now also J1.27 (GPIO12), R2.2, SW10.1, SW2.1
- net key2: now reaches SW11.1
- net key2: now also J1.24 (GPIO13), R3.2, SW3.1, SW7.1
- net key0: now reaches SW9.1
- net key0: now also J1.11 (GPIO9), R1.1, SW1.1, SW5.1
