File: pcbDesign/imModule/inModule.kicad_pcb (KiCad board)
At the start: 2 copper layers, 73 x 50 mm, 10 parts, among them J1 luat-esp32-c3_socket, SW1 SW_DIP_x01, SW2 SW_DIP_x01

Commit message: update inModule pcb add relay holes
Parts:
- removed the REF** at (70.7, 31.3)
- added ?: , , F.Cu at (69.3, 31.3)
- added ?: , , F.Cu at (73.2, 31.3)
- added ?: , , F.Cu at (65.5, 31.3)
- moved REF** 3.03 mm to (61.7, 31.3)
Connections:
- J1 pad 14: unconnected-(J1-GND-Pad14) -> /GND
- J1 pad 16: unconnected-(J1-5V-Pad16) -> /5V
Routing:
- net /GND: track 0.00 -> 59.5 mm, vias 0 -> 2
- net /5V: track 0.00 -> 56.8 mm, vias 0 -> 2
- net /open: track 33.2 -> 38.8 mm
- net Net-(U2-VO+): track 59.3 -> 63.2 mm
- net /lock: track 36.4 -> 40.0 mm
- net Net-(U2-GND): track 108.5 -> 107.2 mm
Other:
- board text added: "+5V"
- board text added: "LOCK"
- board text added: "OPEN"
- board text added: "v0.2.0"

Commit message: uodate inModule change gpio define
Connections:
- J1 pad 23: unconnected-(J1-GPIO07-Pad23) -> /open
- J1 pad 24: /open -> unconnected-(J1-GPIO11-Pad24)
Routing:
- net /open: track 38.8 -> 36.3 mm, vias 0 -> 1
- net unconnected-(J1-GPIO11-Pad24): track 0.00 -> 0.99 mm
Changed lines of the file:
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@@
   (net 16 "unconnected-(J1-GPIO3-Pad20)")
   (net 17 "unconnected-(J1-GPIO10-Pad21)")
-  (net 18 "unconnected-(J1-GPIO07-Pad23)")
+  (net 18 "unconnected-(J1-GPIO11-Pad24)")
   (net 19 "unconnected-(J1-GND-Pad25)")
   (net 20 "unconnected-(J1-3V3-Pad26)")
@@
       (net 29 "/lock") (pinfunction "GPIO06") (pintype "passive"))
     (pad "23" thru_hole oval (at 8.89 -29.31 90) (size 3.39 1.7) (drill 1 (offset 0.845 0)) (layers "*.Cu" "*.Mask")
-      (net 18 "unconnected-(J1-GPIO07-Pad23)") (pinfunction "GPIO07") (pintype "passive+no_connect"))
+      (net 30 "/open") (pinfunction "GPIO07") (pintype "passive"))
     (pad "24" thru_hole oval (at 8.89 -26.77 90) (size 3.39 1.7) (drill 1 (offset 0.845 0)) (layers "*.Cu" "*.Mask")
-      (net 30 "/open") (pinfunction "GPIO11") (pintype "passive"))
+      (net 18 "unconnected-(J1-GPIO11-Pad24)") (pinfunction "GPIO11") (pintype "passive+no_connect"))
     (pad "25" thru_hole oval (at 8.89 -24.23 90) (size 3.39 1.7) (drill 1 (offset 0.845 0)) (layers "*.Cu" "*.Mask")
       (net 19 "unconnected-(J1-GND-Pad25)") (pinfunction "GND") (pintype "passive+no_connect"))
@@
   (segment (start 79.404 37.592) (end 102.616 37.592) (width 0.4) (layer "B.Cu") (net 12))
   (segment (start 73.152 31.34) (end 79.404 37.592) (width 0.4) (layer "B.Cu") (net 12))
+  (segment (start 101.6 32.031522) (end 101.6 32.175) (width 0.5) (layer "F.Cu") (net 18))
+  (segment (start 101.6 32.175) (end 101.6 33.02) (width 0.15) (layer "F.Cu") (net 18))
   (segment (start 101.307107 69.557107) (end 91.44 59.69) (width 0.15) (layer "F.Cu") (net 25))
   (segment (start 77.434214 50.8) (end 83.82 50.8) (width 0.15) (layer "F.Cu") (net 25))
@@
   (segment (start 91.322893 38.217107) (end 96.52 33.02) (width 0.5) (layer "F.Cu") (net 29))
   (arc (start 90.615786 38.51) (mid 90.99847 38.43388) (end 91.322893 38.217107) (width 0.5) (layer "F.Cu") (net 29))
-  (segment (start 67.232 29.64) (end 99.208478 29.64) (width 0.5) (layer "F.Cu") (net 30))
-  (segment (start 65.532 31.34) (end 67.232 29.64) (width 0.5) (layer "F.Cu") (net 30))
-  (segment (start 101.6 32.031522) (end 101.6 32.175) (width 0.5) (layer "F.Cu") (net 30))
-  (segment (start 99.208478 29.64) (end 101.6 32.031522) (width 0.5) (layer "F.Cu") (net 30))
-  (segment (start 101.6 32.175) (end 101.6 33.02) (width 0.15) (layer "F.Cu") (net 30))
+  (segment (start 65.532 31.34) (end 69.752 35.56) (width 0.25) (layer "F.Cu") (net 30))
+  (segment (start 69.752 35.56) (end 85.09 35.56) (width 0.25) (layer "F.Cu") (net 30))
+  (via (at 85.09 35.56) (size 0.8) (drill 0.4) (layers "F.Cu" "B.Cu") (net 30))
+  (segment (start 96.52 35.56) (end 99.06 33.02) (width 0.25) (layer "B.Cu") (net 30))
+  (segment (start 85.09 35.56) (end 96.52 35.56) (width 0.25) (layer "B.Cu") (net 30))
   (segment (start 75.946 47.244) (end 114.046 47.244) (width 0.8) (layer "F.Cu") (net 32))
   (segment (start 69.85 53.34) (end 75.946 47.244) (width 0.8) (layer "F.Cu") (net 32))
